Commit message: grip naming

File: grip_description/urdf/grip.xacro (robot description, xacro)
@@ -26,5 +26,5 @@
   </collision>
 </link>
-<link name="link2_1">
+<link name="link2_1$(arg n)">
   <inertial>
     <origin rpy="0 0 0" xyz="5.153306101393124e-14 0.0 0.011633400273320582"/>
@@ -48,5 +48,5 @@
   </collision>
 </link>
-<link name="_jaw_1">
+<link name="_jaw_1$(arg n)">
   <inertial>
     <origin rpy="0 0 0" xyz="-0.010193902011372998 -0.006835419367933063 0.014639292832342728"/>
@@ -70,5 +70,5 @@
   </collision>
 </link>
-<link name="_jaw_2">
+<link name="_jaw_2$(arg n)">
   <inertial>
     <origin rpy="0 0 0" xyz="0.010193902011372998 0.006835419367933061 0.014639292832342728"/>
@@ -92,5 +92,5 @@
   </collision>
 </link>
-<link name="link1_1">
+<link name="link1_1$(arg n)">
   <inertial>
     <origin rpy="0 0 0" xyz="1.2506577983999133e-15 -7.445092305768896e-16 0.007532920896874856"/>
@@ -116,18 +116,18 @@
 <joint name="j2" type="continuous">
   <origin rpy="0 0 0" xyz="0.0 0.0 0.015"/>
-  <parent link="link1_1"/>
-  <child link="link2_1"/>
+  <parent link="link1_1$(arg n)"/>
+  <child link="link2_1$(arg n)"/>
   <axis xyz="-1.0 0.0 0.0"/>
 </joint>
 <joint name="j3" type="continuous">
   <origin rpy="0 0 0" xyz="0.0 0.009 0.024"/>
-  <parent link="link2_1"/>
-  <child link="_jaw_1"/>
+  <parent link="link2_1$(arg n)"/>
+  <child link="_jaw_1$(arg n)"/>
   <axis xyz="0.0 1.0 0.0"/>
 </joint>
 <joint name="j4" type="continuous">
   <origin rpy="0 0 0" xyz="-0.0 -0.009 0.024"/>
-  <parent link="link2_1"/>
-  <child link="_jaw_2"/>
+  <parent link="link2_1$(arg n)"/>
+  <child link="_jaw_2$(arg n)"/>
   <axis xyz="0.0 1.0 0.0"/>
 </joint>
@@ -135,5 +135,5 @@
   <origin rpy="0 0 0" xyz="0.0 0.0 -0.005"/>
   <parent link="base_link"/>
-  <child link="link1_1"/>
+  <child link="link1_1$(arg n)"/>
   <axis xyz="0.0 0.0 1.0"/>
 </joint>

Commit message: change joint convention

File: grip_description/urdf/grip.xacro (robot description, xacro)
@@ -114,4 +114,11 @@
   </collision>
 </link>
+<link name="distal_wrist_link$(arg n)"/>
+<joint name="j1" type="continuous">
+  <origin rpy="0 0 0" xyz="0.0 0.0 -0.005"/>
+  <parent link="base_link"/>
+  <child link="link1_1$(arg n)"/>
+  <axis xyz="0.0 0.0 1.0"/>
+</joint>
 <joint name="j2" type="continuous">
   <origin rpy="0 0 0" xyz="0.0 0.0 0.015"/>
@@ -121,20 +128,21 @@
 </joint>
 <joint name="j3" type="continuous">
-  <origin rpy="0 0 0" xyz="0.0 0.009 0.024"/>
+  <origin rpy="0 0 0" xyz="0.0 0 0.024"/>
   <parent link="link2_1$(arg n)"/>
+  <child link="distal_wrist_link$(arg n)"/>
+  <axis xyz="0.0 1.0 0.0"/>
+</joint>
+<joint name="j4" type="continuous">
+  <origin rpy="0 0 0" xyz="0.0 0.009 0"/>
+  <parent link="distal_wrist_link$(arg n)"/>
   <child link="_jaw_1$(arg n)"/>
   <axis xyz="0.0 1.0 0.0"/>
 </joint>
-<joint name="j4" type="continuous">
-  <origin rpy="0 0 0" xyz="-0.0 -0.009 0.024"/>
-  <parent link="link2_1$(arg n)"/>
+<joint name="j4b" type="continuous">
+  <origin rpy="0 0 0" xyz="-0.0 -0.009 0"/>
+  <parent link="distal_wrist_link$(arg n)"/>
   <child link="_jaw_2$(arg n)"/>
   <axis xyz="0.0 1.0 0.0"/>
-</joint>
-<joint name="j1" type="continuous">
-  <origin rpy="0 0 0" xyz="0.0 0.0 -0.005"/>
-  <parent link="base_link"/>
-  <child link="link1_1$(arg n)"/>
-  <axis xyz="0.0 0.0 1.0"/>
+  <mimic joint="j4" multiplier="-1.0" offset="0"/>
 </joint>
 </robot>
